Commit message: Various upgrades.

File: sphero_description/urdf/sphero.urdf (robot description, URDF)
Before this commit: robot sphero, 1 links, 0 joints
Links:
- added link base_footprint
- added link imu_link
Joints:
- added joint base_footprint_joint: type fixed, parent base_footprint, child base_link, origin xyz=0 0 0.0381 rpy=0 0 0
- added joint imu_joint: type fixed, parent base_link, child imu_link, origin xyz=0 0 0.0 rpy=0 0 0

Commit message: Updated transform publishing to follow ROS standards more closely (still not fully compliant)

File: sphero_description/urdf/sphero.urdf (robot description, URDF)
Before this commit: robot sphero, 3 links, 2 joints
Joints:
- joint base_footprint_joint: child base_link -> base_footprint; origin xyz=0 0 0.0381 rpy=0 0 0 -> xyz=0 0 -0.0381 rpy=0 0 0; parent base_footprint -> base_link
- joint imu_joint: origin xyz=0 0 0.0 rpy=0 0 0 -> xyz=0 0 0 rpy=0 0 0
